File: KiCad/ADC_BUZZER_OUT.kicad_sch (KiCad schematic)
At the start: 7 parts, among them J10 Conn_01x03, J11 Conn_01x02, U12 ULN2003A

Commit message: new
Parts:
- removed J11: Conn_01x02, Connector_JST:JST_EH_B2B-EH-A_1x02_P2.50mm_Vertical, symbol Connector_Generic:Conn_01x02
- added J11: Conn_01x04, Connector_JST:JST_EH_B4B-EH-A_1x04_P2.50mm_Vertical, symbol Connector_Generic:Conn_01x04
- J10: footprint (none) -> Connector_JST:JST_EH_B3B-EH-A_1x03_P2.50mm_Vertical
Connections:
- net 5V: now also U12.9 (COM), J11.1 (Pin_1), J11.3 (Pin_3)
- net GND: now also J10.1 (Pin_1); no longer J10.3 (Pin_3)
- net at RJ2.1: now also J10.3 (Pin_3); no longer J10.1 (Pin_1)
- net at U12.15 (O2): now also J11.4 (Pin_4)
- net at U12.14 (O3): now also J11.2 (Pin_2)
- no-connect marks 9 -> 8
Changed lines of the file:
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@@
 	(paper "A4")
+	(junction
+		(at 176.53 100.33)
+		(diameter 0)
+		(color 0 0 0 0)
+	)
 	(junction
 		(at 58.42 66.04)
@@
 		(color 0 0 0 0)
 	)
+	(junction
+		(at 199.39 104.14)
+		(diameter 0)
+		(color 0 0 0 0)
+	)
 	(no_connect
 		(at 156.21 118.11)
@@
 	)
 	(no_connect
-		(at 156.21 100.33)
-	)
-	(no_connect
 		(at 135.89 115.57)
 	)
@@
 	(wire
 		(pts
+			(xy 195.58 106.68) (xy 203.2 106.68)
+		)
+		(stroke
+			(width 0)
+			(type default)
+		)
+	)
+	(wire
+		(pts
 			(xy 156.21 105.41) (xy 181.61 105.41)
 		)
@@
 	(wire
 		(pts
+			(xy 194.31 111.76) (xy 203.2 111.76)
+		)
+		(stroke
+			(width 0)
+			(type default)
+		)
+	)
+	(wire
+		(pts
 			(xy 88.9 60.96) (xy 119.38 60.96)
 		)
@@
 	(wire
 		(pts
+			(xy 156.21 107.95) (xy 194.31 107.95)
+		)
+		(stroke
+			(width 0)
+			(type default)
+		)
+	)
+	(wire
+		(pts
+			(xy 194.31 107.95) (xy 194.31 111.76)
+		)
+		(stroke
+			(width 0)
+			(type default)
+		)
+	)
+	(wire
+		(pts
 			(xy 105.41 107.95) (xy 135.89 107.95)
 		)
@@
 	(wire
 		(pts
+			(xy 199.39 109.22) (xy 203.2 109.22)
+		)
+		(stroke
+			(width 0)
+			(type default)
+		)
+	)
+	(wire
+		(pts
 			(xy 176.53 85.09) (xy 176.53 100.33)
 		)
@@
 	(wire
 		(pts
+			(xy 199.39 104.14) (xy 199.39 109.22)
+		)
+		(stroke
+			(width 0)
+			(type default)
+		)
+	)
+	(wire
+		(pts
 			(xy 69.85 57.15) (xy 69.85 63.5)
 		)
@@
 	(wire
 		(pts
+			(xy 195.58 110.49) (xy 195.58 106.68)
+		)
+		(stroke
+			(width 0)
+			(type default)
+		)
+	)
+	(wire
+		(pts
 			(xy 58.42 66.04) (xy 119.38 66.04)
 		)
@@
 	(wire
 		(pts
+			(xy 156.21 110.49) (xy 195.58 110.49)
+		)
+		(stroke
+			(width 0)
+			(type default)
+		)
+	)
+	(wire
+		(pts
 			(xy 88.9 38.1) (xy 88.9 52.07)
 		)
@@
 	(wire
 		(pts
+			(xy 199.39 96.52) (xy 199.39 104.14)
+		)
+		(stroke
+			(width 0)
+			(type default)
+		)
+	)
+	(wire
+		(pts
+			(xy 156.21 100.33) (xy 176.53 100.33)
+		)
+		(stroke
+			(width 0)
+			(type default)
+		)
+	)
+	(wire
+		(pts
 			(xy 69.85 52.07) (xy 69.85 41.91)
 		)
@@
 	(wire
 		(pts
-			(xy 156.21 107.95) (xy 195.58 107.95)
+			(xy 199.39 104.14) (xy 203.2 104.14)
 		)
 		(stroke
@@
 		(pts
 			(xy 66.04 38.1) (xy 58.42 38.1)
-		)
-		(stroke
-			(width 0)
-			(type default)
-		)
-	)
-	(wire
-		(pts
-			(xy 156.21 110.49) (xy 195.58 110.49)
 		)
 		(stroke
@@
 		)
 	)
+	(global_label "5V"
+		(shape input)
+		(at 199.39 96.52 90)
+		(fields_autoplaced yes)
+		(effects
+			(font
+				(size 1.27 1.27)
+			)
+			(justify left)
+		)
+		(property "Intersheetrefs" "${INTERSHEET_REFS}"
+			(at 199.39 91.2367 90)
+			(effects
+				(font
+					(size 1.27 1.27)
+				)
+				(justify left)
+				(hide yes)
+			)
+		)
+	)
 	(hierarchical_label "ADC1"
 		(shape input)
@@
 		(lib_id "Connector_Generic:Conn_01x03")
 		(at 124.46 63.5 0)
+		(mirror x)
 		(unit 1)
 		(exclude_from_sim no)
@@
 		(on_board yes)
 		(dnp no)
-		(fields_autoplaced yes)
 		(property "Reference" "J10"
-			(at 127 62.2299 0)
+			(at 127 64.7701 0)
 			(effects
 				(font
@@
 		)
 		(property "Value" "Conn_01x03"
-			(at 127 64.7699 0)
+			(at 127 62.2301 0)
 			(effects
 				(font
@@
 			)
 		)
-		(property "Footprint" ""
+		(property "Footprint" "Connector_JST:JST_EH_B3B-EH-A_1x03_P2.50mm_Vertical"
 			(at 124.46 63.5 0)
 			(effects
@@
 	)
 	(symbol
-		(lib_id "Connector_Generic:Conn_01x02")
-		(at 200.66 107.95 0)
+		(lib_id "Connector_Generic:Conn_01x04")
+		(at 208.28 106.68 0)
 		(unit 1)
 		(exclude_from_sim no)
@@
 		(fields_autoplaced yes)
 		(property "Reference" "J11"
-			(at 203.2 107.9499 0)
+			(at 210.82 106.6799 0)
 			(effects
 				(font
@@
 			)
 		)
-		(property "Value" "Conn_01x02"
-			(at 203.2 110.4899 0)
+		(property "Value" "Conn_01x04"
+			(at 210.82 109.2199 0)
 			(effects
 				(font
@@
 			)
 		)
-		(property "Footprint" "Connector_JST:JST_EH_B2B-EH-A_1x02_P2.50mm_Vertical"
-			(at 200.66 107.95 0)
+		(property "Footprint" "Connector_JST:JST_EH_B4B-EH-A_1x04_P2.50mm_Vertical"
+			(at 208.28 106.68 0)
 			(effects
 				(font
@@
 		)
 		(property "Datasheet" "~"
-			(at 200.66 107.95 0)
-			(effects
-				(font
-					(size 1.27 1.27)
-				)
-				(hide yes)
-			)
-		)
-		(property "Description" "Generic connector, single row, 01x02, script generated (kicad-library-utils/schlib/autogen/connector/)"
-			(at 200.66 107.95 0)
-			(effects
-				(font
-					(size 1.27 1.27)
-				)
-				(hide yes)
-			)
+			(at 208.28 106.68 0)
+			(effects
+				(font
+					(size 1.27 1.27)
+				)
+				(hide yes)
+			)
+		)
+		(property "Description" "Generic connector, single row, 01x04, script generated (kicad-library-utils/schlib/autogen/connector/)"
+			(at 208.28 106.68 0)
+			(effects
+				(font
+					(size 1.27 1.27)
+				)
+				(hide yes)
+			)
+		)
+		(pin "4"
+		)
+		(pin "2"
+		)
+		(pin "3"
 		)
 		(pin "1"
 		)
-		(pin "2"
-		)
 		(instances
