File: KiCad/CANBUS.kicad_sch (KiCad schematic)
At the start: 6 parts, among them J5 Screw_Terminal_01x02, U5 TJA1051T

Commit message: new
Connections:
- net at J5.2 (Pin_2), R10.1: now also U5.7 (CANH); no longer U5.6 (CANL)
- net at J5.1 (Pin_1), R10.2: now also U5.6 (CANL); no longer U5.7 (CANH)
Other:
- moved on the sheet: R10
Changed lines of the file:
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@@
+	(wire
+		(pts
+			(xy 172.72 101.6) (xy 187.96 101.6)
+		)
+		(stroke
+			(width 0)
+			(type default)
+		)
+	)
 	(wire
 		(pts
@@
 		(pts
 			(xy 187.96 96.52) (xy 187.96 97.79)
-		)
-		(stroke
-			(width 0)
-			(type default)
-		)
-	)
-	(wire
-		(pts
-			(xy 172.72 101.6) (xy 187.96 101.6)
 		)
 		(stroke
@@
 	(symbol
 		(lib_id "Connector:Screw_Terminal_01x02")
-		(at 194.31 97.79 0)
-		(unit 1)
-		(exclude_from_sim no)
-		(in_bom yes)
-		(on_board yes)
-		(dnp no)
-		(fields_autoplaced yes)
+		(at 194.31 100.33 0)
+		(mirror x)
+		(unit 1)
+		(exclude_from_sim no)
+		(in_bom yes)
+		(on_board yes)
+		(dnp no)
 		(property "Reference" "J5"
-			(at 196.85 97.7899 0)
+			(at 196.85 100.3301 0)
 			(effects
 				(font
@@
 		)
 		(property "Value" "Screw_Terminal_01x02"
-			(at 196.85 100.3299 0)
+			(at 196.85 97.7901 0)
 			(effects
 				(font
@@
 		)
 		(property "Footprint" "Connector_Phoenix_MC:PhoenixContact_MC_1,5_2-G-3.81_1x02_P3.81mm_Horizontal"
-			(at 194.31 97.79 0)
+			(at 194.31 100.33 0)
 			(effects
 				(font
@@
 		)
 		(property "Datasheet" "~"
-			(at 194.31 97.79 0)
+			(at 194.31 100.33 0)
 			(effects
 				(font
@@
 		)
 		(property "Description" "Generic screw terminal, single row, 01x02, script generated (kicad-library-utils/schlib/autogen/connector/)"
-			(at 194.31 97.79 0)
+			(at 194.31 100.33 0)
 			(effects
 				(font
@@
 	(symbol
 		(lib_id "Device:R_Small_US")
-		(at 172.72 99.06 180)
+		(at 172.72 99.06 0)
 		(unit 1)
 		(exclude_from_sim no)
@@
 					(size 1.27 1.27)
 				)
-				(justify right)
+				(justify left)
 			)
 		)
@@
 					(size 1.27 1.27)
 				)
-				(justify right)
-			)
-		)
+				(justify left)
+			)
+		)
