File: KiCad/EEPROM.kicad_sch (KiCad schematic)
At the start: 4 parts, among them U8 M24C02-FMN

Commit message: new
Connections:
- no-connect marks 1 -> 0
Changed lines of the file:
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@@
 		(color 0 0 0 0)
-	)
-	(no_connect
-		(at 140.97 81.28)
 	)
 	(wire
