File: KiCad/MCU.kicad_sch (KiCad schematic)
At the start: 20 parts, among them J2 USB_OTG, J3 Conn_01x04, J4 Conn_02x03_Counter_Clockwise, U4 STM32F103C8Tx, Y1 Crystal_Small, Y2 Crystal_Small

Commit message: new
Parts:
- J2: footprint (none) -> Connector_USB:USB_Micro-B_Molex_47346-0001
- Y1: footprint (none) -> Crystal:Crystal_SMD_HC49-SD
- Y2: footprint (none) -> Crystal:Crystal_C26-LF_D2.1mm_L6.5mm_Horizontal
- renumbered U4 to U1
Connections:
- net BOOT0: now also R6.1
- net BOOT1: no longer R6.1
Other:
- moved on the sheet: Y1
Changed lines of the file:
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@@
 	(wire
 		(pts
-			(xy 240.03 57.15) (xy 240.03 60.96)
+			(xy 240.03 58.42) (xy 240.03 60.96)
 		)
 		(stroke
@@
 	(wire
 		(pts
+			(xy 240.03 53.34) (xy 240.03 52.07)
+		)
+		(stroke
+			(width 0)
+			(type default)
+		)
+	)
+	(wire
+		(pts
 			(xy 205.74 24.13) (xy 205.74 29.21)
 		)
@@
 	(wire
 		(pts
+			(xy 59.69 46.99) (xy 85.09 46.99)
+		)
+		(stroke
+			(width 0)
+			(type default)
+		)
+	)
+	(wire
+		(pts
 			(xy 259.08 60.96) (xy 240.03 60.96)
 		)
@@
 	(wire
 		(pts
-			(xy 59.69 46.99) (xy 85.09 46.99)
-		)
-		(stroke
-			(width 0)
-			(type default)
-		)
-	)
-	(wire
-		(pts
 			(xy 205.74 39.37) (xy 198.12 39.37)
 		)
@@
 		)
 	)
-	(global_label "D_N"
+	(global_label "3V3"
 		(shape input)
-		(at 85.09 46.99 0)
+		(at 198.12 19.05 90)
 		(fields_autoplaced yes)
 		(effects
@@
 		)
 		(property "Intersheetrefs" "${INTERSHEET_REFS}"
-			(at 91.6433 46.99 0)
+			(at 198.12 12.5572 90)
 			(effects
 				(font
@@
 		)
 	)
-	(global_label "3V3"
+	(global_label "BOOT0"
 		(shape input)
-		(at 198.12 19.05 90)
+		(at 114.3 53.34 180)
 		(fields_autoplaced yes)
 		(effects
@@
 				(size 1.27 1.27)
 			)
-			(justify left)
+			(justify right)
 		)
 		(property "Intersheetrefs" "${INTERSHEET_REFS}"
-			(at 198.12 12.5572 90)
+			(at 105.2067 53.34 0)
 			(effects
 				(font
 					(size 1.27 1.27)
 				)
-				(justify left)
+				(justify right)
 				(hide yes)
 			)
 		)
 	)
-	(global_label "BOOT0"
+	(global_label "D_N"
 		(shape input)
-		(at 114.3 53.34 180)
+		(at 85.09 46.99 0)
 		(fields_autoplaced yes)
 		(effects
@@
 				(size 1.27 1.27)
 			)
-			(justify right)
+			(justify left)
 		)
 		(property "Intersheetrefs" "${INTERSHEET_REFS}"
-			(at 105.2067 53.34 0)
+			(at 91.6433 46.99 0)
 			(effects
 				(font
 					(size 1.27 1.27)
 				)
-				(justify right)
+				(justify left)
 				(hide yes)
 			)
@@
 		)
 	)
-	(global_label "BOOT1"
+	(global_label "BOOT0"
 		(shape input)
 		(at 229.87 114.3 180)
@@
 			)
 		)
-		(property "Footprint" ""
+		(property "Footprint" "Crystal:Crystal_C26-LF_D2.1mm_L6.5mm_Horizontal"
 			(at 240.03 73.66 0)
 			(effects
@@
 		(dnp no)
 		(fields_autoplaced yes)
-		(property "Reference" "U4"
+		(property "Reference" "U1"
 			(at 140.5733 121.92 0)
 			(effects
@@
 			(project ""
 				(path "/5dc221ca-bb86-41f1-a15e-48a3ea813131/651630f0-d7fb-4f36-b717-d65930401c84"
-					(reference "U4")
+					(reference "U1")
 					(unit 1)
 				)
@@
 	(symbol
 		(lib_id "Device:Crystal_Small")
-		(at 240.03 54.61 90)
+		(at 240.03 55.88 90)
 		(unit 1)
 		(exclude_from_sim no)
@@
 		(fields_autoplaced yes)
 		(property "Reference" "Y1"
-			(at 242.57 53.3399 90)
+			(at 242.57 54.6099 90)
 			(effects
 				(font
@@
 		)
 		(property "Value" "Crystal_Small"
-			(at 242.57 55.8799 90)
+			(at 242.57 57.1499 90)
 			(effects
 				(font
@@
 			)
 		)
-		(property "Footprint" ""
-			(at 240.03 54.61 0)
+		(property "Footprint" "Crystal:Crystal_SMD_HC49-SD"
+			(at 240.03 55.88 0)
 			(effects
 				(font
@@
 		)
 		(property "Datasheet" "~"
-			(at 240.03 54.61 0)
+			(at 240.03 55.88 0)
 			(effects
 				(font
@@
 		)
 		(property "Description" "Two pin crystal, small symbol"
-			(at 240.03 54.61 0)
+			(at 240.03 55.88 0)
 			(effects
 				(font
@@
 			)
 		)
-		(property "Footprint" ""
+		(property "Footprint" "Connector_USB:USB_Micro-B_Molex_47346-0001"
 			(at 55.88 45.72 0)
 			(effects
