File: KiCad/PWM.kicad_sch (KiCad schematic)
At the start: 5 parts, among them J9 Conn_01x06

Commit message: new
Connections:
- net GND: now also D6.1 (RK), D6.2 (GK), D6.3 (BK); no longer D6.4 (BA), D6.5 (GA), D6.6 (RA)
- net PWM2: now also J9.1 (Pin_1); no longer J9.5 (Pin_5)
- net PWM3: now also J9.5 (Pin_5); no longer J9.1 (Pin_1)
- net at R32.2: now also D6.4 (BA); no longer D6.1 (RK)
- net at R33.2: now also D6.5 (GA); no longer D6.2 (GK)
- net at R34.2: now also D6.6 (RA); no longer D6.3 (BK)
Other:
- moved on the sheet: D6
Changed lines of the file:
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@@
-	)
-	(junction
-		(at 160.02 101.6)
-		(diameter 0)
-		(color 0 0 0 0)
-	)
-	(junction
-		(at 149.86 91.44)
-		(diameter 0)
-		(color 0 0 0 0)
 	)
 	(junction
@@
 		(color 0 0 0 0)
 	)
+	(junction
+		(at 149.86 101.6)
+		(diameter 0)
+		(color 0 0 0 0)
+	)
+	(junction
+		(at 160.02 91.44)
+		(diameter 0)
+		(color 0 0 0 0)
+	)
 	(wire
 		(pts
@@
 	(wire
 		(pts
+			(xy 149.86 73.66) (xy 149.86 101.6)
+		)
+		(stroke
+			(width 0)
+			(type default)
+		)
+	)
+	(wire
+		(pts
 			(xy 144.78 96.52) (xy 154.94 96.52)
 		)
@@
 	(wire
 		(pts
-			(xy 144.78 101.6) (xy 160.02 101.6)
-		)
-		(stroke
-			(width 0)
-			(type default)
-		)
-	)
-	(wire
-		(pts
-			(xy 144.78 91.44) (xy 149.86 91.44)
-		)
-		(stroke
-			(width 0)
-			(type default)
-		)
-	)
-	(wire
-		(pts
-			(xy 149.86 91.44) (xy 179.07 91.44)
-		)
-		(stroke
-			(width 0)
-			(type default)
-		)
-	)
-	(wire
-		(pts
-			(xy 160.02 101.6) (xy 166.37 101.6)
+			(xy 144.78 101.6) (xy 149.86 101.6)
+		)
+		(stroke
+			(width 0)
+			(type default)
+		)
+	)
+	(wire
+		(pts
+			(xy 144.78 91.44) (xy 160.02 91.44)
 		)
 		(stroke
@@
 	(wire
 		(pts
+			(xy 160.02 91.44) (xy 179.07 91.44)
+		)
+		(stroke
+			(width 0)
+			(type default)
+		)
+	)
+	(wire
+		(pts
+			(xy 160.02 73.66) (xy 160.02 91.44)
+		)
+		(stroke
+			(width 0)
+			(type default)
+		)
+	)
+	(wire
+		(pts
 			(xy 177.8 96.52) (xy 186.69 96.52)
 		)
@@
 	(wire
 		(pts
-			(xy 149.86 73.66) (xy 149.86 91.44)
+			(xy 149.86 101.6) (xy 166.37 101.6)
 		)
 		(stroke
@@
 		(pts
 			(xy 196.85 101.6) (xy 214.63 101.6)
-		)
-		(stroke
-			(width 0)
-			(type default)
-		)
-	)
-	(wire
-		(pts
-			(xy 160.02 73.66) (xy 160.02 101.6)
 		)
 		(stroke
@@
 	(symbol
 		(lib_id "Device:LED_RGB")
-		(at 191.77 96.52 0)
+		(at 191.77 96.52 180)
 		(unit 1)
 		(exclude_from_sim no)
@@
 		(fields_autoplaced yes)
 		(property "Reference" "D6"
-			(at 191.77 82.55 0)
+			(at 191.77 83.82 0)
 			(effects
 				(font
@@
 		)
 		(property "Value" "LED_RGB"
-			(at 191.77 85.09 0)
+			(at 191.77 86.36 0)
 			(effects
 				(font
@@
 		)
 		(property "Footprint" "LED_SMD:LED_RGB_5050-6"
-			(at 191.77 97.79 0)
+			(at 191.77 95.25 0)
 			(effects
 				(font
@@
 		)
 		(property "Datasheet" "~"
-			(at 191.77 97.79 0)
-			(effects
-				(font
+			(at 191.77 95.25 0)
+			(effects
+				(font
