File: KiCad/RS485.kicad_sch (KiCad schematic)
At the start: 11 parts, among them J7 RJ45_USER, J8 Conn_01x04, U11 MAX485E

Commit message: new
Connections:
- net 5V: now also R29.1; no longer R29.2
- net GND: now also R30.2; no longer R30.1
- net at J7.3, U11.6 (A): now also R28.2, R30.1; no longer R28.1, R30.2
- net at J7.5, U11.7 (B): now also R28.1, R29.2; no longer R28.2, R29.1
Other:
- moved on the sheet: R28, R29, R30
Changed lines of the file:
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@@
 	(text "RX TX GND 5V"
 		(exclude_from_sim no)
-		(at 110.236 23.368 0)
+		(at 91.44 24.13 0)
 		(effects
 			(font
@@
 	(symbol
 		(lib_id "Device:R_Small_US")
-		(at 160.02 67.31 0)
+		(at 160.02 67.31 180)
 		(unit 1)
 		(exclude_from_sim no)
@@
 					(size 1.27 1.27)
 				)
-				(justify left)
+				(justify right)
 			)
 		)
@@
 					(size 1.27 1.27)
 				)
-				(justify left)
+				(justify right)
 			)
 		)
@@
 	(symbol
 		(lib_id "Device:R_Small_US")
-		(at 160.02 82.55 0)
+		(at 160.02 82.55 180)
 		(unit 1)
 		(exclude_from_sim no)
@@
 					(size 1.27 1.27)
 				)
-				(justify left)
+				(justify right)
 			)
 		)
@@
 					(size 1.27 1.27)
 				)
-				(justify left)
+				(justify right)
 			)
 		)
@@
 	(symbol
 		(lib_id "Device:R_Small_US")
-		(at 160.02 53.34 0)
+		(at 160.02 53.34 180)
 		(unit 1)
 		(exclude_from_sim no)
@@
 					(size 1.27 1.27)
 				)
-				(justify left)
+				(justify right)
 			)
 		)
@@
 					(size 1.27 1.27)
 				)
-				(justify left)
-			)
-		)
+				(justify right)
+			)
+		)
