File: KiCad/SDCARD.kicad_sch (KiCad schematic)
At the start: 13 parts, among them U10 TVS_5V, U9 SDCARD_KLS

Commit message: new
Connections:
- net SPI_SD_DETECT: no longer R22.1, U10.3 (IO3)
- net SPI_SD_MISO: no longer U10.1 (IO1)
- net at R21.2, U9.9 (DETECT_SDCARD): now also R22.1, U10.3 (IO3)
- net at R20.2, U9.7 (MISO/DAT0): now also U10.1 (IO1)
Other:
- moved on the sheet: R20, R21
Changed lines of the file:
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@@
-	(wire
-		(pts
-			(xy 132.08 96.52) (xy 142.24 96.52)
-		)
-		(stroke
-			(width 0)
-			(type default)
-		)
-	)
 	(wire
 		(pts
@@
 	(wire
 		(pts
-			(xy 83.82 96.52) (xy 92.71 96.52)
+			(xy 83.82 96.52) (xy 85.09 96.52)
 		)
 		(stroke
@@
 	(wire
 		(pts
-			(xy 124.46 88.9) (xy 142.24 88.9)
+			(xy 99.06 88.9) (xy 100.33 88.9)
 		)
 		(stroke
@@
 	(wire
 		(pts
+			(xy 110.49 48.26) (xy 110.49 54.61)
+		)
+		(stroke
+			(width 0)
+			(type default)
+		)
+	)
+	(wire
+		(pts
+			(xy 129.54 54.61) (xy 129.54 81.28)
+		)
+		(stroke
+			(width 0)
+			(type default)
+		)
+	)
+	(wire
+		(pts
+			(xy 101.6 114.3) (xy 100.33 114.3)
+		)
+		(stroke
+			(width 0)
+			(type default)
+		)
+	)
+	(wire
+		(pts
+			(xy 101.6 76.2) (xy 110.49 76.2)
+		)
+		(stroke
+			(width 0)
+			(type default)
+		)
+	)
+	(wire
+		(pts
 			(xy 92.71 96.52) (xy 97.79 96.52)
 		)
@@
 	(wire
 		(pts
-			(xy 110.49 48.26) (xy 110.49 54.61)
-		)
-		(stroke
-			(width 0)
-			(type default)
-		)
-	)
-	(wire
-		(pts
-			(xy 129.54 54.61) (xy 129.54 81.28)
-		)
-		(stroke
-			(width 0)
-			(type default)
-		)
-	)
-	(wire
-		(pts
-			(xy 101.6 114.3) (xy 100.33 114.3)
-		)
-		(stroke
-			(width 0)
-			(type default)
-		)
-	)
-	(wire
-		(pts
-			(xy 101.6 76.2) (xy 110.49 76.2)
-		)
-		(stroke
-			(width 0)
-			(type default)
-		)
-	)
-	(wire
-		(pts
 			(xy 100.33 88.9) (xy 100.33 114.3)
 		)
@@
 	(wire
 		(pts
+			(xy 90.17 96.52) (xy 92.71 96.52)
+		)
+		(stroke
+			(width 0)
+			(type default)
+		)
+	)
+	(wire
+		(pts
 			(xy 119.38 54.61) (xy 119.38 62.23)
 		)
@@
 	(wire
 		(pts
-			(xy 97.79 96.52) (xy 127 96.52)
-		)
-		(stroke
-			(width 0)
-			(type default)
-		)
-	)
-	(wire
-		(pts
 			(xy 83.82 76.2) (xy 96.52 76.2)
 		)
@@
 	(wire
 		(pts
+			(xy 100.33 88.9) (xy 142.24 88.9)
+		)
+		(stroke
+			(width 0)
+			(type default)
+		)
+	)
+	(wire
+		(pts
 			(xy 139.7 54.61) (xy 139.7 62.23)
 		)
@@
 	(wire
 		(pts
-			(xy 100.33 88.9) (xy 119.38 88.9)
-		)
-		(stroke
-			(width 0)
-			(type default)
-		)
-	)
-	(wire
-		(pts
 			(xy 116.84 119.38) (xy 125.73 119.38)
 		)
@@
 	(wire
 		(pts
-			(xy 83.82 88.9) (xy 100.33 88.9)
+			(xy 83.82 88.9) (xy 93.98 88.9)
 		)
 		(stroke
@@
 		(pts
 			(xy 137.16 93.98) (xy 137.16 102.87)
+		)
+		(stroke
+			(width 0)
+			(type default)
+		)
+	)
+	(wire
+		(pts
+			(xy 97.79 96.52) (xy 142.24 96.52)
 		)
 		(stroke
@@
 	(symbol
 		(lib_id "Device:R_Small_US")
-		(at 129.54 96.52 90)
+		(at 87.63 96.52 90)
 		(unit 1)
 		(exclude_from_sim no)
@@
 		(fields_autoplaced yes)
 		(property "Reference" "R21"
-			(at 129.54 90.17 90)
+			(at 87.63 90.17 90)
 			(effects
 				(font
@@
 		)
 		(property "Value" "1K8"
-			(at 129.54 92.71 90)
+			(at 87.63 92.71 90)
 			(effects
 				(font
@@
 		)
 		(property "Footprint" "Resistor_SMD:R_0805_2012Metric_Pad1.20x1.40mm_HandSolder"
-			(at 129.54 96.52 0)
+			(at 87.63 96.52 0)
 			(effects
 				(font
@@
 		)
 		(property "Datasheet" "~"
-			(at 129.54 96.52 0)
+			(at 87.63 96.52 0)
 			(effects
 				(font
@@
 		)
 		(property "Description" "Resistor, small US symbol"
-			(at 129.54 96.52 0)
+			(at 87.63 96.52 0)
 			(effects
 				(font
@@
 	(symbol
 		(lib_id "Device:R_Small_US")
-		(at 121.92 88.9 90)
+		(at 96.52 88.9 90)
 		(unit 1)
 		(exclude_from_sim no)
@@
 		(fields_autoplaced yes)
 		(property "Reference" "R20"
-			(at 121.92 82.55 90)
+			(at 96.52 82.55 90)
 			(effects
 				(font
@@
 		)
 		(property "Value" "47R"
-			(at 121.92 85.09 90)
+			(at 96.52 85.09 90)
 			(effects
 				(font
@@
 		)
 		(property "Footprint" "Resistor_SMD:R_0805_2012Metric_Pad1.20x1.40mm_HandSolder"
-			(at 121.92 88.9 0)
+			(at 96.52 88.9 0)
 			(effects
 				(font
@@
 		)
 		(property "Datasheet" "~"
-			(at 121.92 88.9 0)
+			(at 96.52 88.9 0)
 			(effects
 				(font
@@
 		)
 		(property "Description" "Resistor, small US symbol"
-			(at 121.92 88.9 0)
-			(effects
-				(font
+			(at 96.52 88.9 0)
+			(effects
+				(font
