File: KiCad/SIM800C.kicad_sch (KiCad schematic)
At the start: 19 parts, among them J12 SIM_Card-8066, Q1 BC337, U13 SIM800C

Commit message: new
Connections:
- net 3V7: now also R40.2; no longer R40.1
- net CLK_SIM: now also R38.2; no longer R38.1
- net DATA_SIM: now also R39.2; no longer R39.1
- net GND: now also Q1.3 (E), R41.2; no longer Q1.2 (B), R40.2, R41.1
- net RESET_SIM: now also R37.2; no longer R37.1
- net at D7.2 (A): now also R35.1; no longer R35.2
- net at J12.2 (RST): now also R37.1; no longer R37.2
- net at J12.3 (CLK): now also R38.1; no longer R38.2
- net at J12.7 (I/O): now also R39.1; no longer R39.2
- net at U13.42 (STATUS): now also R35.2; no longer R35.1
- new net: Q1.2 (B), R40.1, R41.1
Other:
- moved on the sheet: R35, R37, R38, R39, R40, R41
Changed lines of the file:
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@@
+	(wire
+		(pts
+			(xy 77.47 100.33) (xy 77.47 107.95)
+		)
+		(stroke
+			(width 0)
+			(type default)
+		)
+	)
 	(wire
 		(pts
@@
 	(wire
 		(pts
-			(xy 77.47 87.63) (xy 77.47 107.95)
+			(xy 77.47 87.63) (xy 77.47 95.25)
 		)
 		(stroke
@@
 	(wire
 		(pts
-			(xy 88.9 101.6) (xy 88.9 107.95)
-		)
-		(stroke
-			(width 0)
-			(type default)
-		)
-	)
-	(wire
-		(pts
 			(xy 208.28 26.67) (xy 208.28 30.48)
 		)
@@
 	(wire
 		(pts
-			(xy 88.9 92.71) (xy 88.9 96.52)
+			(xy 88.9 92.71) (xy 88.9 107.95)
 		)
 		(stroke
@@
 	(symbol
 		(lib_id "Device:R_Small_US")
-		(at 88.9 99.06 180)
+		(at 77.47 97.79 0)
 		(unit 1)
 		(exclude_from_sim no)
@@
 		(fields_autoplaced yes)
 		(property "Reference" "R41"
-			(at 91.44 97.7899 0)
-			(effects
-				(font
-					(size 1.27 1.27)
-				)
-				(justify right)
+			(at 80.01 96.5199 0)
+			(effects
+				(font
+					(size 1.27 1.27)
+				)
+				(justify left)
 			)
 		)
 		(property "Value" "4K7"
-			(at 91.44 100.3299 0)
-			(effects
-				(font
-					(size 1.27 1.27)
-				)
-				(justify right)
+			(at 80.01 99.0599 0)
+			(effects
+				(font
+					(size 1.27 1.27)
+				)
+				(justify left)
 			)
 		)
 		(property "Footprint" "Resistor_SMD:R_0805_2012Metric_Pad1.20x1.40mm_HandSolder"
-			(at 88.9 99.06 0)
+			(at 77.47 97.79 0)
 			(effects
 				(font
@@
 		)
 		(property "Datasheet" "~"
-			(at 88.9 99.06 0)
+			(at 77.47 97.79 0)
 			(effects
 				(font
@@
 		)
 		(property "Description" "Resistor, small US symbol"
-			(at 88.9 99.06 0)
+			(at 77.47 97.79 0)
 			(effects
 				(font
@@
 	(symbol
 		(lib_id "Device:R_Small_US")
-		(at 68.58 87.63 90)
+		(at 68.58 87.63 270)
 		(unit 1)
 		(exclude_from_sim no)
@@
 	(symbol
 		(lib_id "Device:R_Small_US")
-		(at 114.3 149.86 90)
+		(at 114.3 149.86 270)
 		(unit 1)
 		(exclude_from_sim no)
@@
 	(symbol
 		(lib_id "Device:R_Small_US")
-		(at 121.92 152.4 90)
+		(at 121.92 152.4 270)
 		(unit 1)
 		(exclude_from_sim no)
@@
 	(symbol
 		(lib_id "Device:R_Small_US")
-		(at 198.12 87.63 90)
+		(at 198.12 87.63 270)
 		(unit 1)
 		(exclude_from_sim no)
@@
 	(symbol
 		(lib_id "Device:R_Small_US")
-		(at 129.54 160.02 90)
-		(unit 1)
-		(exclude_from_sim no)
+		(at 129.54 160.02 270)
+		(unit 1)
+		(exclude_from_sim no)
