File: KiCad/SPI1.kicad_sch (KiCad schematic)
At the start: 8 parts, among them J6 Conn_01x05, U6 74HC14_, U7 TVS_5V

Commit message: new
Parts:
- removed F4, F5: RESETTABLE_FUSE-0603, My_Library:RESETTABLE_FUSE-0603, symbol User_Libraries:RESETTABLE_FUSE
- added Q2: BSS138, Package_TO_SOT_SMD:SOT-23, symbol Transistor_FET:BSS138
- added R42, R47: 10K, Resistor_SMD:R_0805_2012Metric_Pad1.20x1.40mm_HandSolder, symbol Device:R_Small_US
Connections:
- net 5V: now also J6.1 (Pin_1), R47.2; no longer F1.1
- net GND: now also J6.2 (Pin_2); no longer F2.1
- net MISO: now also F1.1, Q2.3 (D), R47.1; no longer F3.1, U6.8 (4Y)
- net MOSI_: now also F2.1
- net SCLK: now also F3.1
- net SPI1_MISO: now also Q2.2 (S), R42.1; no longer U6.5 (3A)
- net at F2.2: now also J6.4 (Pin_4); no longer J6.2 (Pin_2)
- net at F3.2: now also J6.5 (Pin_5); no longer J6.3 (Pin_3)
- net at F1.2: now also J6.3 (Pin_3); no longer J6.1 (Pin_1)
- net 3Y: no longer names the net of U6.6 (3Y)
- net 3Y: no longer U6.9 (4A)
- new net 3V3: Q2.1 (G), R42.2
- no-connect marks 1 -> 5
Other:
- moved on the sheet: F1, F2, F3
